Commit message: Updated FIne tuned parameters

File: urdf/truck_urdf.urdf.xacro (robot description, xacro)
@@ -66,5 +66,5 @@
       <surface>
         <contact><ode><kp>1e6</kp><kd>1.0</kd><max_vel>0.2</max_vel><min_depth>0.001</min_depth></ode></contact>
-        <friction><ode><mu>1.2</mu><mu2>1.2</mu2><slip1>0.01</slip1><slip2>0.0</slip2></ode></friction>
+        <friction><ode><mu>3.2</mu><mu2>3.2</mu2><slip1>0.01</slip1><slip2>0.0</slip2></ode></friction>
       </surface>
     </collision>
@@ -108,5 +108,5 @@
       <surface>
         <contact><ode><kp>1e6</kp><kd>1.0</kd><max_vel>0.2</max_vel><min_depth>0.001</min_depth></ode></contact>
-        <friction><ode><mu>1.2</mu><mu2>1.2</mu2><slip1>0.01</slip1><slip2>0.0</slip2></ode></friction>
+        <friction><ode><mu>3.2</mu><mu2>3.2</mu2><slip1>0.01</slip1><slip2>0.0</slip2></ode></friction>
       </surface>
     </collision>
@@ -133,5 +133,5 @@
       <surface>
         <contact><ode><kp>1e6</kp><kd>1.0</kd><max_vel>0.2</max_vel><min_depth>0.001</min_depth></ode></contact>
-        <friction><ode><mu>1.2</mu><mu2>1.2</mu2><slip1>0.01</slip1><slip2>0.0</slip2></ode></friction>
+        <friction><ode><mu>7.2</mu><mu2>7.2</mu2><slip1>0.01</slip1><slip2>0.0</slip2></ode></friction>
       </surface>
     </collision>
@@ -157,5 +157,5 @@
       <surface>
         <contact><ode><kp>1e6</kp><kd>1.0</kd><max_vel>0.2</max_vel><min_depth>0.001</min_depth></ode></contact>
-        <friction><ode><mu>1.2</mu><mu2>1.2</mu2><slip1>0.01</slip1><slip2>0.0</slip2></ode></friction>
+        <friction><ode><mu>7.2</mu><mu2>7.2</mu2><slip1>0.01</slip1><slip2>0.0</slip2></ode></friction>
       </surface>
     </collision>
@@ -172,5 +172,5 @@
     <inertial>
       <origin xyz="3.69323682747336E-10 0.571256988776015 0.117353006753824" rpy="0 0 0"/>
-      <mass value="15.484741148508"/>
+      <mass value="95.484741148508"/>
       <inertia ixx="13.6421910845191" ixy="-2.48524307383535E-09" ixz="6.24243486154171E-09"
                iyy="4.71963963467751"  iyz="0.00663582007885279"  izz="15.5438252225012"/>
@@ -275,5 +275,5 @@
     <inertial>
       <origin xyz="3.6686853555068E-10 0.571256988777377 0.117353006753846" rpy="0 0 0"/>
-      <mass value="15.484741148483"/>
+      <mass value="95.484741148483"/>
       <inertia ixx="13.6421910845091" ixy="-2.52925029141024E-09" ixz="6.24522738612748E-09"
                iyy="4.71963963467603"  iyz="0.00663582007955939"  izz="15.5438252224907"/>
